Commit message: add new urdf

File: assets/urdf/panda_isaac/robots/franka_panda_stick_copy.urdf (robot description, URDF)
Before this commit: robot panda, 14 links, 13 joints
Links:
- removed link base_link
- removed link base_link_x
- removed link base_link_y
- removed link world
- link panda_ee_finger: mass 0.1 -> None
- link panda_ee_tip: mass 0.01 -> None
- link panda_link0: mass 2.92 -> None
- link panda_link1: mass 2.74 -> None
- link panda_link2: mass 2.74 -> None
- link panda_link3: mass 2.38 -> None
- link panda_link4: mass 2.38 -> None
- link panda_link5: mass 2.74 -> None
- link panda_link6: mass 1.55 -> None
- link panda_link7: mass 0.54 -> None
Joints:
- removed joint omni_joint_theta
- removed joint omni_joint_x
- removed joint omni_joint_y
- removed joint panda_joint_base
